Commit message: Now pluto is runnable.

File: pluto_description/urdf/pluto.urdf.xacro (robot description, xacro)
@@ -4,8 +4,9 @@
   xmlns:controller="http://playerstage.sourceforge.net/gazebo/xmlschema/#controller"
   xmlns:interface="http://playerstage.sourceforge.net/gazebo/xmlschema/#interface"
+  xmlns:sensor="http://playerstage.sourceforge.net/gazebo/xmlschema/#sensor"
   name="pluto">
   <xacro:include filename="$(find uos_common_urdf)/common.xacro" />
   <xacro:include filename="$(find uos_common_urdf)/urdf/imu.gazebo.urdf.xacro" />
-  <xacro:include filename="$(find pluto_description)/urdf/rotunit.urdf.xacro" />
+  <xacro:include filename="$(find rotunit)/urdf/rotunit.urdf.xacro" />
   <xacro:property name="M_PI" value="3.14159265359"/>
   <xacro:property name="imu_stdev" value="0.00017" />
@@ -83,5 +84,6 @@
   </link>
   <joint name="base_footprint_to_base_joint" type="fixed">
-    <origin xyz="0 0 0.2" rpy="0 ${-M_PI/18.0} 0" />
+    <!-- origin xyz="0 0 0.2" rpy="0 ${-M_PI/18.0} 0" /-->
+    <origin xyz="0 0 0.2" rpy="0 0 0" />
     <parent link="base_footprint"/>
     <child link="base_link" />
@@ -133,5 +135,5 @@
   <!--Wheel Macro-->
   <xacro:macro name="wheel" params="name parent xyz">
-    <link name="wheel_${name}">
+    <link name="${name}_link">
       <visual>
         <origin xyz="0 0 0" rpy="0 0 0" />
@@ -157,5 +159,5 @@
       <origin xyz="${xyz}" rpy="0 0 0"/>
       <parent link="${parent}"/>
-      <child link="wheel_${name}"/>
+      <child link="${name}_link"/>
       <axis xyz="0 1 0"/>
     </joint>
@@ -203,5 +205,5 @@
             ${imu_offset_y}
             ${imu_offset_z}"
-      rpy="0 0 0" />
+      rpy="${M_PI} 0 ${M_PI/2.0}" />
   </joint>
   <!-- inertial measurement unit for gazebo -->
@@ -248,3 +250,17 @@
     </plugin>
   </gazebo>
+  <xacro:macro name="simple_transmission" params="name">
+    <transmission name="${name}_trans">
+      <type>transmission_interface/SimpleTransmission</type>
+      <joint name="${name}_joint">
+        <hardwareInterface>EffortJointInterface</hardwareInterface>
+      </joint>
+      <actuator name="${name}_motor">
+        <hardwareInterface>EffortJointInterface</hardwareInterface>
+        <mechanicalReduction>1</mechanicalReduction>
+      </actuator>
+    </transmission>
+  </xacro:macro>
+  <xacro:simple_transmission name="virtual_left_to_base" />
+  <xacro:simple_transmission name="virtual_right_to_base" />
 </robot>

Commit message: simplified meshes for collision

File: pluto_description/urdf/pluto.urdf.xacro (robot description, xacro)
@@ -74,5 +74,5 @@
       <origin xyz="0 0 0" rpy="0 0 0" />
       <geometry>
-        <mesh filename="package://pluto_description/meshes/pluto_base.stl"/>
+        <mesh filename="package://pluto_description/meshes/pluto_base_collision.stl"/>
       </geometry>
     </collision>
@@ -148,5 +148,6 @@
         <origin xyz="0 0 0" rpy="0 0 0" />
         <geometry>
-          <mesh filename="package://pluto_description/meshes/pluto_wheel.stl"/>
+          <mesh
+          filename="package://pluto_description/meshes/pluto_wheel_collision.stl"/>
         </geometry>
       </collision>

Commit message: added pluto lever collision mesh

File: pluto_description/urdf/pluto.urdf.xacro (robot description, xacro)
@@ -104,5 +104,5 @@
         <origin xyz="0 0 0" rpy="0 0 ${rot}" />
         <geometry>
-          <mesh filename="package://pluto_description/meshes/pluto_lever.stl"/>
+          <mesh filename="package://pluto_description/meshes/pluto_lever_collision.stl"/>
         </geometry>
       </collision>

Commit message: changed urdf

File: pluto_description/urdf/pluto.urdf.xacro (robot description, xacro)
@@ -53,6 +53,6 @@
   <xacro:property name="axis_length" value="0.47" />
   <xacro:property name="turning_adaptation" value="0.95" />
-  <xacro:property name="body_mass" value="0.1"/>
-  <xacro:property name="wheel_mass" value="0.01"/>
+  <xacro:property name="body_mass" value="40.0"/>
+  <xacro:property name="wheel_mass" value="3.0"/>
   <xacro:property name="wheel_radius" value="0.15"/>
   <xacro:property name="wheel_thickness" value="0.065"/>
@@ -142,5 +142,5 @@
         </geometry>
         <material name="black" >
-          <color rgba="0.3 0.3 0.3 1" />
+          <color rgba="0 0 0 1" />
         </material>
       </visual>
@@ -163,4 +163,12 @@
       <axis xyz="0 1 0"/>
     </joint>
+    <gazebo reference="${name}_link">
+      <mu1>1</mu1>
+      <mu2>1</mu2>
+      <material>Gazebo/Black</material>
+      <kp>10000000</kp>
+      <kd>10</kd>
+      <selfCollide>false</selfCollide>
+    </gazebo>
   </xacro:macro>
   <xacro:wheel

Commit message: added velodyne to urdf

File: pluto_description/urdf/pluto.urdf.xacro (robot description, xacro)
@@ -34,4 +34,11 @@
   <xacro:property name="rotunit_offset_z"
     value="${body_height/2-0.014 + rotunit_box_z/2}"/>
+  <xacro:property name="velodyne_height" value="0.1442"/>
+  <xacro:property name="velodyne_radius" value="0.04265"/>
+  <xacro:property name="velodyne_height_to_lense" value="0.090805"/>
+  <xacro:property name="velodyne_offset_x" value="${body_length/2 - 0.0265 + 0.02}"/>
+  <xacro:property name="velodyne_offset_y" value="0"/>
+  <xacro:property name="velodyne_offset_z"
+    value="${-0.005 + velodyne_height/2}"/>
   <xacro:property name="virtual_axis_left_offset_x"
     value="${body_length/2 - pannel_depth-bearing_pos_wheel_2_3
@@ -218,4 +225,24 @@
   <!-- inertial measurement unit for gazebo -->
   <xacro:imu_gazebo link="imu" imu_topic="imu/data" update_rate="100.0" stdev="${imu_stdev}" />
+  <link name="velodyne">
+    <visual>
+      <origin xyz="0 0 ${-velodyne_height_to_lense}" rpy="0 0 0" />
+      <geometry>
+        <cylinder length="0.1442" radius="0.04265"/>
+      </geometry>
+      <material name="silver">
+        <color rgba="0.5 0.5 0.5 1" />
+      </material>
+    </visual>
+  </link>
+  <joint name="velodyne_to_base_joint" type="fixed">
+    <child link="velodyne" />
+    <parent link="base_link" />
+    <origin
+      xyz=" ${velodyne_offset_x}
+            ${velodyne_offset_y}
+            ${velodyne_offset_z + velodyne_height_to_lense}"
+      rpy="0 0 0" />
+  </joint>
   <joint name="rotunit_to_base_joint" type="fixed">
     <child link="rotunit_box_link" />

Commit message: changed gazebo map and dirty fixed urdf

File: pluto_description/urdf/pluto.urdf.xacro (robot description, xacro)
@@ -120,5 +120,5 @@
         mass="${horizontal_lever_mass}"/>
     </link>
-    <joint name="virtual_${side}_to_base_joint" type="revolute">
+    <joint name="virtual_${side}_to_base_joint" type="fixed">
       <origin xyz="${xyz}"/>
       <axis xyz="0 1 0"/>
@@ -254,4 +254,18 @@
       rpy="0 0 ${-M_PI/2}" />
   </joint>
+  <!-- GPS Sensor -->
+  <gazebo>
+    <plugin name="novatel_gps_sim" filename="libhector_gazebo_ros_gps.so">
+      <alwaysOn>1</alwaysOn>
+      <updateRate>10.0</updateRate>
+      <bodyName>base_footprint</bodyName>
+      <topicName>gps/fix</topicName>
+      <velocityTopicName>gps/fix_velocity</velocityTopicName>
+      <drift>0.5 0.5 0.5</drift>
+      <gaussianNoise>0.1 0.1 0.1</gaussianNoise>
+      <velocityDrift>0 0 0</velocityDrift>
+      <velocityGaussianNoise>0.1 0.1 0.1</velocityGaussianNoise>
+    </plugin>
+   </gazebo>
   <gazebo>
     <plugin name="volksbot_diffdrive" filename="libgazebo_ros_diffdrive_uos.so">

Commit message: chnaged for riegl laser scanner

File: pluto_description/urdf/pluto.urdf.xacro (robot description, xacro)
@@ -8,5 +8,5 @@
   <xacro:include filename="$(find uos_common_urdf)/common.xacro" />
   <xacro:include filename="$(find uos_common_urdf)/urdf/imu.gazebo.urdf.xacro" />
-  <xacro:include filename="$(find uos_rotunit_driver)/urdf/rotunit.urdf.xacro" />
+  <xacro:include filename="$(find riegl_vline_driver)/urdf/riegl_vz400i_mount.urdf.xacro" />
   <xacro:property name="M_PI" value="3.14159265359"/>
   <xacro:property name="imu_stdev" value="0.00017" />
@@ -28,10 +28,10 @@
   <xacro:property name="pannel_height" value="0.09"/>
   <xacro:property name="pannel_depth" value="0.082"/>
-  <xacro:property name="rotunit_offset_x"
-    value="${body_width/2 - 0.1 - 0.19/2 + rotunit_box_x/2}"/>
-  <xacro:property name="rotunit_offset_y"
+  <xacro:property name="riegl_vz400i_offset_x"
+    value="${body_width/2 - 0.1}"/>
+  <xacro:property name="riegl_vz400i_offset_y"
     value="0"/>
-  <xacro:property name="rotunit_offset_z"
-    value="${body_height/2-0.014 + rotunit_box_z/2}"/>
+  <xacro:property name="riegl_vz400i_offset_z"
+    value="${body_height/2-0.014 + 0.012}"/>
   <xacro:property name="velodyne_height" value="0.1442"/>
   <xacro:property name="velodyne_radius" value="0.04265"/>
@@ -245,12 +245,12 @@
       rpy="0 0 0" />
   </joint>
-  <joint name="rotunit_to_base_joint" type="fixed">
-    <child link="rotunit_box_link" />
+  <joint name="riegl_vz400i_to_base_joint" type="fixed">
+    <child link="riegl_mount_base" />
     <parent link="base_link" />
     <origin
-      xyz=" ${rotunit_offset_x}
-            ${rotunit_offset_y}
-            ${rotunit_offset_z}"
-      rpy="0 0 ${-M_PI/2}" />
+      xyz=" ${riegl_vz400i_offset_x}
+            ${riegl_vz400i_offset_y}
+            ${riegl_vz400i_offset_z}"
+      rpy="0 0 0" />
   </joint>
   <gazebo>

Commit message: added modified imu joints to urdf

File: pluto_description/urdf/pluto.urdf.xacro (robot description, xacro)
@@ -64,7 +64,13 @@
   <xacro:property name="wheel_radius" value="0.15"/>
   <xacro:property name="wheel_thickness" value="0.065"/>
-  <xacro:property name="imu_offset_x" value="${body_length/2 - 0.285}"/>
-  <xacro:property name="imu_offset_y" value="0"/>
-  <xacro:property name="imu_offset_z" value="${- body_height/2 + 0.03}"/>
+  <xacro:property name="imu_center_offset_x" value="${body_length/2 - 0.285}"/>
+  <xacro:property name="imu_center_offset_y" value="0"/>
+  <xacro:property name="imu_center_offset_z" value="${- body_height/2 + 0.03}"/>
+  <xacro:property name="imu_left_offset_x" value="0.1"/>
+  <xacro:property name="imu_left_offset_y" value="0.2"/>
+  <xacro:property name="imu_left_offset_z" value="0.05"/>
+  <xacro:property name="imu_right_offset_x" value="0.1"/>
+  <xacro:property name="imu_right_offset_y" value="-0.2"/>
+  <xacro:property name="imu_right_offset_z" value="0.05"/>
   <link name="base_footprint"/>
   <link name="base_link">
@@ -203,5 +209,5 @@
     parent="base_link"
     xyz="-0.23 -0.19 ${(-body_height/2.0)+(bearing_height/2.0)}" />
-  <link name="imu">
+  <link name="imu_center">
     <visual>
       <origin xyz="0 0 0" rpy="0 0 0" />
@@ -214,12 +220,54 @@
     </visual>
   </link>
-  <joint name="imu_to_base_joint" type="fixed">
-    <parent link="base_link" />
-    <child link="imu" />
-    <origin
-      xyz=" ${imu_offset_x}
-            ${imu_offset_y}
-            ${imu_offset_z}"
-      rpy="${M_PI} 0 ${M_PI/2.0}" />
+  <joint name="imu_center_to_base_joint" type="fixed">
+    <parent link="base_link" />
+    <child link="imu_center" />
+    <origin
+      xyz=" ${imu_center_offset_x}
+            ${imu_center_offset_y}
+            ${imu_center_offset_z}"
+      rpy="${M_PI} -0.1660595 ${M_PI/2.0}" />
+   <!-- rpy="${M_PI} 0 ${M_PI/2.0}" /> -->
+  </joint>
+  <link name="imu_left">
+    <visual>
+      <origin xyz="0 0 0" rpy="0 0 0" />
+      <geometry>
+        <box size="0.06 0.06 0.02"/>
+      </geometry>
+      <material name="white" >
+        <color rgba="0.8 0.8 0.8 1" />
+      </material>
+    </visual>
+  </link>
+  <!-- phidgets driver solution for left to right handed coordinates : multiply a -1 to every axis -->
+  <joint name="imu_left_to_base_joint" type="fixed">
+    <parent link="base_link" />
+    <child link="imu_left" />
+    <origin
+      xyz=" ${imu_left_offset_x}
+            ${imu_left_offset_y}
+            ${imu_left_offset_z}"
+            rpy="0 ${M_PI/2.0} ${-M_PI/2.0}" />
+  </joint>
+  <link name="imu_right">
+    <visual>
+      <origin xyz="0 0 0" rpy="0 0 0" />
+      <geometry>
+        <box size="0.06 0.06 0.02"/>
+      </geometry>
+      <material name="white" >
+        <color rgba="0.8 0.8 0.8 1" />
+      </material>
+    </visual>
+  </link>
+  <joint name="imu_right_to_base_joint" type="fixed">
+    <parent link="base_link" />
+    <child link="imu_right" />
+    <origin
+      xyz=" ${imu_right_offset_x}
+            ${imu_right_offset_y}
+            ${imu_right_offset_z}"
+            rpy="0 ${-M_PI/2.0} ${-M_PI/2.0}" />
   </joint>
   <!-- inertial measurement unit for gazebo -->

Commit message: removed trailing whitespaces and changed some rotations. not tested

File: pluto_description/urdf/pluto.urdf.xacro (robot description, xacro)
@@ -10,4 +10,5 @@
   <xacro:include filename="$(find riegl_driver)/urdf/riegl_vz400i_mount.urdf.xacro" />
   <xacro:property name="M_PI" value="3.14159265359"/>
+  <xacro:property name="footprint_to_base_rpy_p" value="-0.1660595"/>
   <xacro:property name="imu_stdev" value="0.00017" />
   <xacro:property name="body_height" value="0.21"/>
@@ -98,5 +99,5 @@
   <joint name="base_footprint_to_base_joint" type="fixed">
     <!-- origin xyz="0 0 0.2" rpy="0 ${-M_PI/18.0} 0" /-->
-    <origin xyz="0 0 0.2" rpy="0 0 0" />
+    <origin xyz="0 0 0.2" rpy="0 ${footprint_to_base_rpy_p} 0" />
     <parent link="base_footprint"/>
     <child link="base_link" />
@@ -227,6 +228,6 @@
             ${imu_center_offset_y}
             ${imu_center_offset_z}"
-      rpy="${M_PI} -0.1660595 ${M_PI/2.0}" />
-   <!-- rpy="${M_PI} 0 ${M_PI/2.0}" /> -->
+      rpy="${M_PI} ${-footprint_to_base_rpy_p} ${M_PI/2.0}" />
+   <!-- TODO: test -->
   </joint>
   <link name="imu_left">
@@ -291,5 +292,5 @@
             ${velodyne_offset_y}
             ${velodyne_offset_z + velodyne_height_to_lense}"
-      rpy="0 0 0" />
+      rpy="0 ${-M_PI/22} 0" />
   </joint>
   <joint name="riegl_vz400i_to_base_joint" type="fixed">

Commit message: tested params

File: pluto_description/urdf/pluto.urdf.xacro (robot description, xacro)
@@ -10,5 +10,5 @@
   <xacro:include filename="$(find riegl_driver)/urdf/riegl_vz400i_mount.urdf.xacro" />
   <xacro:property name="M_PI" value="3.14159265359"/>
-  <xacro:property name="footprint_to_base_rpy_p" value="-0.1660595"/>
+  <xacro:property name="footprint_to_base_rpy_p" value="-0.12"/>
   <xacro:property name="imu_stdev" value="0.00017" />
   <xacro:property name="body_height" value="0.21"/>
@@ -228,5 +228,5 @@
             ${imu_center_offset_y}
             ${imu_center_offset_z}"
-      rpy="${M_PI} ${-footprint_to_base_rpy_p} ${M_PI/2.0}" />
+            rpy="${M_PI} 0 ${M_PI/2.0}" />
    <!-- TODO: test -->
   </joint>
@@ -292,5 +292,5 @@
             ${velodyne_offset_y}
             ${velodyne_offset_z + velodyne_height_to_lense}"
-      rpy="0 ${-M_PI/22} 0" />
+      rpy="0 0 0" />
   </joint>
   <joint name="riegl_vz400i_to_base_joint" type="fixed">

Commit message: added back rotation to wheel axis

File: pluto_description/urdf/pluto.urdf.xacro (robot description, xacro)
@@ -128,5 +128,6 @@
     </link>
     <joint name="virtual_${side}_to_base_joint" type="revolute">
-      <origin xyz="${xyz}"/>
+      <origin xyz="${xyz}"
+        rpy="0 ${-footprint_to_base_rpy_p} 0" />
       <axis xyz="0 1 0"/>
       <limit effort="1000" lower="-0.4" upper="0.4" velocity="10"/>
@@ -135,4 +136,5 @@
     </joint>
   </xacro:macro>
+  <!-- set initial rot to  footprint_to_base_rpy_p -->
   <xacro:virtual_axis
     side="left"

Commit message: added correct joint between virtual_axis_X and imu_X with X element of [left,right]

File: pluto_description/urdf/pluto.urdf.xacro (robot description, xacro)
@@ -246,11 +246,9 @@
   <!-- phidgets driver solution for left to right handed coordinates : multiply a -1 to every axis -->
   <joint name="imu_left_to_base_joint" type="fixed">
-    <parent link="base_link" />
+    <parent link="virtual_axis_left" />
     <child link="imu_left" />
     <origin
-      xyz=" ${imu_left_offset_x}
-            ${imu_left_offset_y}
-            ${imu_left_offset_z}"
-            rpy="0 ${M_PI/2.0} ${-M_PI/2.0}" />
+      xyz="0 0 0.2"
+      rpy="0 0 0" />
   </joint>
   <link name="imu_right">
@@ -266,11 +264,9 @@
   </link>
   <joint name="imu_right_to_base_joint" type="fixed">
-    <parent link="base_link" />
+    <parent link="virtual_axis_right" />
     <child link="imu_right" />
     <origin
-      xyz=" ${imu_right_offset_x}
-            ${imu_right_offset_y}
-            ${imu_right_offset_z}"
-            rpy="0 ${-M_PI/2.0} ${-M_PI/2.0}" />
+      xyz="0 0 0.2"
+      rpy="0 0 0" />
   </joint>
   <!-- inertial measurement unit for gazebo -->

Commit message: Revert "Merge branch 'update-urdf' into 'master'"
This reverts merge request !18

File: pluto_description/urdf/pluto.urdf.xacro (robot description, xacro)
@@ -128,6 +128,5 @@
     </link>
     <joint name="virtual_${side}_to_base_joint" type="revolute">
-      <origin xyz="${xyz}"
-        rpy="0 ${-footprint_to_base_rpy_p} 0" />
+      <origin xyz="${xyz}"/>
       <axis xyz="0 1 0"/>
       <limit effort="1000" lower="-0.4" upper="0.4" velocity="10"/>
@@ -136,5 +135,4 @@
     </joint>
   </xacro:macro>
-  <!-- set initial rot to  footprint_to_base_rpy_p -->
   <xacro:virtual_axis
     side="left"
@@ -246,9 +244,11 @@
   <!-- phidgets driver solution for left to right handed coordinates : multiply a -1 to every axis -->
   <joint name="imu_left_to_base_joint" type="fixed">
-    <parent link="virtual_axis_left" />
+    <parent link="base_link" />
     <child link="imu_left" />
     <origin
-      xyz="0 0 0.2"
-      rpy="0 0 0" />
+      xyz=" ${imu_left_offset_x}
+            ${imu_left_offset_y}
+            ${imu_left_offset_z}"
+            rpy="0 ${M_PI/2.0} ${-M_PI/2.0}" />
   </joint>
   <link name="imu_right">
@@ -264,9 +264,11 @@
   </link>
   <joint name="imu_right_to_base_joint" type="fixed">
-    <parent link="virtual_axis_right" />
+    <parent link="base_link" />
     <child link="imu_right" />
     <origin
-      xyz="0 0 0.2"
-      rpy="0 0 0" />
+      xyz=" ${imu_right_offset_x}
+            ${imu_right_offset_y}
+            ${imu_right_offset_z}"
+            rpy="0 ${-M_PI/2.0} ${-M_PI/2.0}" />
   </joint>
   <!-- inertial measurement unit for gazebo -->

Commit message: fix covariance params

File: pluto_description/urdf/pluto.urdf.xacro (robot description, xacro)
@@ -10,5 +10,5 @@
   <xacro:include filename="$(find riegl_driver)/urdf/riegl_vz400i_mount.urdf.xacro" />
   <xacro:property name="M_PI" value="3.14159265359"/>
-  <xacro:property name="footprint_to_base_rpy_p" value="-0.12"/>
+  <xacro:property name="footprint_to_base_rpy_p" value="-0.143"/>
   <xacro:property name="imu_stdev" value="0.00017" />
   <xacro:property name="body_height" value="0.21"/>

Commit message: update laserscan direction

File: pluto_description/urdf/pluto.urdf.xacro (robot description, xacro)
@@ -10,5 +10,5 @@
   <xacro:include filename="$(find riegl_driver)/urdf/riegl_vz400i_mount.urdf.xacro" />
   <xacro:property name="M_PI" value="3.14159265359"/>
-  <xacro:property name="footprint_to_base_rpy_p" value="-0.143"/>
+  <xacro:property name="footprint_to_base_rpy_p" value="-0.142"/>
   <xacro:property name="imu_stdev" value="0.00017" />
   <xacro:property name="body_height" value="0.21"/>

Commit message: old params

File: pluto_description/urdf/pluto.urdf.xacro (robot description, xacro)
@@ -128,5 +128,6 @@
     </link>
     <joint name="virtual_${side}_to_base_joint" type="revolute">
-      <origin xyz="${xyz}"/>
+      <origin xyz="${xyz}"
+        rpy="0 ${-footprint_to_base_rpy_p} 0" />
       <axis xyz="0 1 0"/>
       <limit effort="1000" lower="-0.4" upper="0.4" velocity="10"/>
@@ -135,4 +136,5 @@
     </joint>
   </xacro:macro>
+  <!-- set initial rot to  footprint_to_base_rpy_p -->
   <xacro:virtual_axis
     side="left"
@@ -244,11 +246,9 @@
   <!-- phidgets driver solution for left to right handed coordinates : multiply a -1 to every axis -->
   <joint name="imu_left_to_base_joint" type="fixed">
-    <parent link="base_link" />
+    <parent link="virtual_axis_left" />
     <child link="imu_left" />
     <origin
-      xyz=" ${imu_left_offset_x}
-            ${imu_left_offset_y}
-            ${imu_left_offset_z}"
-            rpy="0 ${M_PI/2.0} ${-M_PI/2.0}" />
+      xyz="0 0 0.2"
+      rpy="0 0 0" />
   </joint>
   <link name="imu_right">
@@ -264,11 +264,9 @@
   </link>
   <joint name="imu_right_to_base_joint" type="fixed">
-    <parent link="base_link" />
+    <parent link="virtual_axis_right" />
     <child link="imu_right" />
     <origin
-      xyz=" ${imu_right_offset_x}
-            ${imu_right_offset_y}
-            ${imu_right_offset_z}"
-            rpy="0 ${-M_PI/2.0} ${-M_PI/2.0}" />
+      xyz="0 0 0.2"
+      rpy="0 0 0" />
   </joint>
   <!-- inertial measurement unit for gazebo -->
